File: Air.kicad_pcb (KiCad board)
At the start: 2 copper layers, 101 parts, among them J1 AIR1, J10 USB_C_Receptacle_USB2.0_14P, J11 Conn_ST_STDC14, J12 CAN, J13 CAN, J2 AIR2, J3 AIR3, J4 AIR4, J5 AIR5, J6 AIR6, J7 AIR7, J8 AIR8, J9 24V IN, Q1 2SC2712, Q2 2SC2712, Q3 2SC2712, Q4 2SC2712, Q5 2SC2712, Q6 2SC2712, Q7 2SC2712, Q8 2SC2712, SW1 NRST, U1 TLP293, U10 CH340E, U11 STM32F303K8Tx, U12 TJA1441, U2 TLP293, U3 TLP293, U4 TLP293, U5 TLP293, U6 TLP293, U7 TLP293, U8 TLP293, U9 NJM12877

Commit message: chore: Update Air.kicad_pro configuration file
Parts:
- added J12: CANR, Connector_PinHeader_2.54mm:PinHeader_1x02_P2.54mm_Vertical, F.Cu at (297.8, 258.4)
- added REF**: MountingHole_3.2mm_M3, MountingHole:MountingHole_3.2mm_M3, F.Cu at (276.0, 282.0)
- added REF**: MountingHole_3.2mm_M3, MountingHole:MountingHole_3.2mm_M3, F.Cu at (276.0, 233.0)
- added REF**: MountingHole_3.2mm_M3, MountingHole:MountingHole_3.2mm_M3, F.Cu at (361.0, 282.0)
- added REF**: MountingHole_3.2mm_M3, MountingHole:MountingHole_3.2mm_M3, F.Cu at (361.0, 233.0)
- D11, D21, D31, D41, D51, D61, D71, D81: moved to B.Cu
- U11: moved to F.Cu
- moved Q5 364.3 mm to (348.3, 350.2)
- moved R61 361.1 mm to (340.6, 360.4), turned to -90 degrees
- moved R51 359.0 mm to (349.5, 360.4), turned to -90 degrees
- moved R54 357.4 mm to (348.3, 347.7)
- moved R53 357.2 mm to (344.4, 347.7)
- moved Q6 354.8 mm to (339.4, 350.2)
- moved R81 351.0 mm to (322.9, 360.4), turned to -90 degrees
- moved D51 350.5 mm to (347.0, 340.1)
- moved R62 347.9 mm to (335.6, 350.2), turned to -90 degrees
- moved R71 347.8 mm to (331.7, 360.4), turned to -90 degrees
- moved R74 346.6 mm to (330.5, 347.7)
- moved R52 345.9 mm to (344.4, 350.2), turned to -90 degrees
- moved Q7 345.3 mm to (330.5, 350.2)
- moved R64 344.1 mm to (339.4, 347.7)
- moved R63 343.8 mm to (335.6, 347.7)
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- renumbered J12 to J13, J13 to J14
Connections:
- net Net-(J12-Pin_3) renamed /CANL
- J13 pad 4: Net-(J12-Pin_4) -> /CANH
- J14 pad 4: Net-(J12-Pin_4) -> /CANH
- R8 pad 1: Net-(J12-Pin_4) -> Net-(J12-Pin_2)
- U12 pad 7: Net-(J12-Pin_4) -> /CANH
Routing:
- net +3V3: track 0.00 -> 109.1 mm, vias 0 -> 6
- net +5V: track 0.00 -> 97.8 mm, vias 0 -> 2
- net +24V: track 0.00 -> 93.0 mm, vias 0 -> 11
- net GNDPWR: track 0.00 -> 74.4 mm, vias 0 -> 9
- net /NRST: track 0.00 -> 64.7 mm, vias 0 -> 1
- net /VCP_TX: track 0.00 -> 46.9 mm, vias 0 -> 2
- net /CANH: track 0.00 -> 39.4 mm, vias 0 -> 1
- net /CANL: track 0.00 -> 39.3 mm, vias 0 -> 1
- net /VCP_RX: track 0.00 -> 37.9 mm, vias 0 -> 2
- net /SWO: track 0.00 -> 34.1 mm, vias 0 -> 1
- net /Drive/GPIO4: track 0.00 -> 31.4 mm
- net /Drive/GPIO2: track 0.00 -> 26.8 mm
- net /Drive/GPIO1: track 0.00 -> 25.7 mm
- net Net-(U10-UD+): track 0.00 -> 25.0 mm
- net Net-(U10-UD-): track 0.00 -> 24.3 mm, vias 0 -> 2
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- added copper zone on B.Cu, net GND
- added copper zone on F.Cu, net GND
- added copper zone on B.Cu, net GNDPWR
- added copper zone on F.Cu, net GNDPWR
Other:
- board outline added: 91 x 55 mm
