File: Air.kicad_sch (KiCad schematic)
At the start: 10 parts

Commit message: chore: Initial commit
Parts:
- removed D?: SS2040FL, symbol Device:D_Schottky_Small_Filled
- added D? (x4): SS2040FL, symbol Device:D_Schottky_Filled
- added J? (x3): OUT1, symbol Connector_Generic:Conn_01x02
- added J?: SWD, symbol Connector_Generic:Conn_01x06
- added U?: STM32F303K8Tx, Package_QFP:LQFP-32_7x7mm_P0.8mm, symbol MCU_ST_STM32F3:STM32F303K8Tx
Connections:
- net +24V: now also D?.1 (K), D?.1 (K), D?.1 (K), D?.1 (K), J?.2 (Pin_2), J?.2 (Pin_2), J?.2 (Pin_2)
- net GND: now also J?.3 (Pin_3)
- net OUT1: now also D?.2 (A), D?.2 (A), D?.2 (A), D?.2 (A), J?.1 (Pin_1), J?.1 (Pin_1), J?.1 (Pin_1)
- new net NRST: J?.5 (Pin_5)
- new net SWCLK: J?.2 (Pin_2)
- new net SWDIO: J?.4 (Pin_4)
- new net SWO: J?.6 (Pin_6)
- new net VCC: J?.1 (Pin_1)

Commit message: chore: Update Air.kicad_pro configuration file
Parts:
- removed D? (x3): SS2040FL, symbol Device:D_Schottky_Filled
- removed J? (x3): OUT1, symbol Connector_Generic:Conn_01x02
- removed J?: SWD, symbol Connector_Generic:Conn_01x06
- added C1, C2, C3, C4, C5: 0.1u, symbol Device:C
- added C6: 10u, symbol Device:C
- added D1: AIR1, symbol Device:LED
- added D12, D13, D14, D15, D16, D17, D18: SS2040FL, symbol Device:D_Schottky_Filled
- added D2: AIR2, symbol Device:LED
- added D3: AIR3, symbol Device:LED
- added D4: AIR4, symbol Device:LED
- added D5: AIR5, symbol Device:LED
- added D6: AIR6, symbol Device:LED
- added D7: AIR7, symbol Device:LED
- added D8: AIR8, symbol Device:LED
- added J10: Conn_ST_STDC14, symbol Connector:Conn_ST_STDC14
- added J11: CAN, symbol Connector_Generic:Conn_01x04
- added J12: USB_C_Receptacle, symbol Connector:USB_C_Receptacle
- added J2: AIR2, symbol Connector_Generic:Conn_01x02
- added J3: AIR3, symbol Connector_Generic:Conn_01x02
- added J4: AIR4, symbol Connector_Generic:Conn_01x02
- added J5: AIR5, symbol Connector_Generic:Conn_01x02
- added J6: AIR6, symbol Connector_Generic:Conn_01x02
- added J7: AIR7, symbol Connector_Generic:Conn_01x02
- added J8: AIR8, symbol Connector_Generic:Conn_01x02
- added J9: 24V IN, symbol Connector_Generic:Conn_01x02
- added R1, R2, R3, R4, R5, R6, R7, R8: R, symbol Device:R
- added R10: 10k, symbol Device:R
- added R2A, R2B, R2C, R2D: 120, symbol Device:R
- added R9: 10k (DNP), symbol Device:R
- added SW1: NRST, symbol Switch:SW_Push
- added U2: TLP291-4, Package_SO:SOIC-16_4.55x10.3mm_P1.27mm, symbol Isolator:TLP291-4
- added U4: LD1117S33TR, Package_TO_SOT_SMD:SOT-223-3_TabPin2, symbol Regulator_Linear:LD1117S33TR_SOT223
- J1: renamed from J?; value OUT1 -> AIR1
- gave numbers to parts that had none: 7
Connections:
- net +24V: now also D1.2 (A), D12.1 (K), D13.1 (K), D14.1 (K), D15.1 (K), D16.1 (K), D17.1 (K), D18.1 (K), D2.2 (A), D3.2 (A), D4.2 (A), D5.2 (A), D6.2 (A), D7.2 (A), D8.2 (A), J2.2 (Pin_2), J3.2 (Pin_2), J4.2 (Pin_2), J5.2 (Pin_2), J6.2 (Pin_2), J7.2 (Pin_2), J8.2 (Pin_2), J9.2 (Pin_2)
- net GND: now also U3.16 (VSS), U3.32 (VSS), C1.2, C2.2, C3.2, C4.2, C5.2, C6.2, J10.5 (GND), J10.7 (GND), J11.1 (Pin_1), R10.2, R2A.1, R2B.1, R2C.1, R2D.1, SW1.1, U4.1 (GND)
- net GNDPWR: now also J9.1 (Pin_1), U2.11, U2.13, U2.15, U2.9
- net NRST: now also U3.4 (NRST), C1.1, J10.12 (~{RST}), SW1.2
- net OUT1: now also R1.2
- net OUT2: now also D12.2 (A), J2.1 (Pin_1), R2.2
- net OUT3: now also D13.2 (A), J3.1 (Pin_1), R3.2; no longer U1.10
- net SWCLK: now also U3.24 (PA14), J10.6 (JCLK/SWCLK)
- net SWDIO: now also U3.23 (PA13), J10.4 (JTMS/SWDIO)
- net SWO: now also U3.26 (PB3), J10.8 (JTDO/SWO)
- net +3V3: now reaches U3.1 (VDD)
- net +3V3: now also U3.17 (VDD), U3.5 (VDDA), C2.1, C3.1, C4.1, C6.1, J10.3 (VCC), R9.1, U4.2 (VO)
- net CAN_RX: now reaches U3.21 (PA11)
- net CAN_TX: now reaches U3.22 (PA12)
- net VCP_RX: now reaches U3.25 (PA15)
- net VCP_RX: now also J10.13 (VCP_RX)
- net at U3.31 (BOOT0): now also R10.1, R9.2
- net VCP_TX: now reaches U3.8 (PA2)
- net VCP_TX: now also J10.14 (VCP_TX)
- new net: J12.A1 (GND), J12.A12 (GND), J12.B1 (GND), J12.B12 (GND)
- new net: J12.A4 (VBUS), J12.A9 (VBUS), J12.B4 (VBUS), J12.B9 (VBUS)
- new net: D8.1 (K), R8.1
- new net: R2C.2, U2.6
- new net: D4.1 (K), R4.1
- new net: D6.1 (K), R6.1
- new net: D3.1 (K), R3.1
- new net: R2A.2, U2.2
- new net: D5.1 (K), R5.1
- new net: R2B.2, U2.4
- new net: D1.1 (K), R1.1
- new net: D7.1 (K), R7.1
- new net: R2D.2, U2.8
- new net: D2.1 (K), R2.1
- new net +5V: C5.1, J11.2 (Pin_2), U4.3 (VI)
- new net CANH: J11.4 (Pin_4)
- new net CANL: J11.3 (Pin_3)
- new net GPIO5: U2.1
- new net GPIO6: U2.3
- new net GPIO7: U2.5
- new net GPIO8: U2.7
- new net OUT4: D14.2 (A), J4.1 (Pin_1), R4.2, U1.10
- new net OUT5: D15.2 (A), J5.1 (Pin_1), R5.2, U2.16
- new net OUT6: D16.2 (A), J6.1 (Pin_1), R6.2, U2.14
- new net OUT7: D17.2 (A), J7.1 (Pin_1), R7.2, U2.12
- new net OUT8: D18.2 (A), J8.1 (Pin_1), R8.2, U2.10
- no-connect marks 0 -> 21
Other:
- moved on the sheet: D11, J1, R1A, R1B, R1C, R1D, U1A, U1B, U1C, U1D, U3

Commit message: Update Air.kicad_pro configuration file
Parts:
- removed D12, D13, D14, D15, D16, D17, D18: SS2040FL, symbol Device:D_Schottky_Filled
- removed D2: AIR2, symbol Device:LED
- removed D4: AIR4, symbol Device:LED
- removed D5: AIR5, symbol Device:LED
- removed D6: AIR6, symbol Device:LED
- removed D7: AIR7, symbol Device:LED
- removed D8: AIR8, symbol Device:LED
- removed J12: USB_C_Receptacle, symbol Connector:USB_C_Receptacle
- removed R1A, R1B, R1C, R1D, R2A, R2B, R2C, R2D: 120, symbol Device:R
- removed R2, R8: R, symbol Device:R
- removed U1, U2: TLP291-4, Package_SO:SOIC-16_4.55x10.3mm_P1.27mm, symbol Isolator:TLP291-4
- added C10: 0.1u, Capacitor_SMD:C_0603_1608Metric_Pad1.08x0.95mm_HandSolder, symbol Device:C
- added C9: 220u, Capacitor_SMD:CP_Elec_8x10, symbol Device:C
- added D21, D31, D41, D51, D61, D71, D81: SS2040FL, Diode_SMD:D_SOD-123F, symbol Device:D_Schottky_Filled
- added D22: AIR2, Diode_SMD:D_0603_1608Metric_Pad1.05x0.95mm_HandSolder, symbol Device:LED
- added D32: AIR3, Diode_SMD:D_0603_1608Metric_Pad1.05x0.95mm_HandSolder, symbol Device:LED
- added D42: AIR4, Diode_SMD:D_0603_1608Metric_Pad1.05x0.95mm_HandSolder, symbol Device:LED
- added D52: AIR5, Diode_SMD:D_0603_1608Metric_Pad1.05x0.95mm_HandSolder, symbol Device:LED
- added D62: AIR6, Diode_SMD:D_0603_1608Metric_Pad1.05x0.95mm_HandSolder, symbol Device:LED
- added D72: AIR7, Diode_SMD:D_0603_1608Metric_Pad1.05x0.95mm_HandSolder, symbol Device:LED
- added D82: AIR8, Diode_SMD:D_0603_1608Metric_Pad1.05x0.95mm_HandSolder, symbol Device:LED
- added J10: USB_C_Receptacle_USB2.0_14P, symbol Connector:USB_C_Receptacle_USB2.0_14P
- added Q1, Q2, Q3, Q4, Q5, Q6, Q7, Q8: 2SC2712, Package_TO_SOT_SMD:SC-59_Handsoldering, symbol Device:Q_NPN_BEC
- added R11, R12, R14, R21, R22, R23, R24, R31, R32, R33, R34, R41, R42, R43, R44, R51, R52, R53, R54, R61, R62, R63, R64, R71, R72, R73, R74, R81, R82, R83, R84: 10k, Resistor_SMD:R_0603_1608Metric_Pad0.98x0.95mm_HandSolder, symbol Device:R
- added U1, U2, U3, U4, U5, U6, U7, U8: TLP293, Package_SO:SOIC-4_4.55x2.6mm_P1.27mm, symbol Isolator:TLP293
- added U10: CH340E, Package_SO:MSOP-10_3x3mm_P0.5mm, symbol Interface_USB:CH340E
- added U12: MCP2562-E-MF, Package_DFN_QFN:DFN-8-1EP_3x3mm_P0.65mm_EP1.55x2.4mm, symbol Interface_CAN_LIN:MCP2562-E-MF
- C1, C2, C3, C4, C5: footprint (none) -> Capacitor_SMD:C_0603_1608Metric_Pad1.08x0.95mm_HandSolder
- C6: value 10u -> 0.1u; footprint (none) -> Capacitor_SMD:C_0603_1608Metric_Pad1.08x0.95mm_HandSolder
- D11: footprint (none) -> Diode_SMD:D_SOD-123F
- D12: renamed from D1; footprint (none) -> Diode_SMD:D_0603_1608Metric_Pad1.05x0.95mm_HandSolder
- D3: value AIR3 -> POWER; footprint (none) -> Diode_SMD:D_0603_1608Metric_Pad1.05x0.95mm_HandSolder
- J1, J2, J3, J4, J5, J6, J7, J8: footprint (none) -> Connector_JST:JST_XH_S2B-XH-A_1x02_P2.50mm_Horizontal
- J9: footprint (none) -> Connector_AMASS:AMASS_XT60PW-M_1x02_P7.20mm_Horizontal
- R1: renamed from R9; footprint (none) -> Resistor_SMD:R_0603_1608Metric_Pad0.98x0.95mm_HandSolder
- R13: renamed from R1; value R -> 10k; footprint (none) -> Resistor_SMD:R_0603_1608Metric_Pad0.98x0.95mm_HandSolder
- R2: renamed from R10; footprint (none) -> Resistor_SMD:R_0603_1608Metric_Pad0.98x0.95mm_HandSolder
- R3: value R -> 1k; footprint (none) -> Resistor_SMD:R_0603_1608Metric_Pad0.98x0.95mm_HandSolder
- R4, R5, R6, R7: value R -> 10k; footprint (none) -> Resistor_SMD:R_0603_1608Metric_Pad0.98x0.95mm_HandSolder
- renumbered J10 to J11, J11 to J12, U3 to U11, U4 to U9
Connections:
- net +24V: now also C9.1, D21.1 (K), D22.2 (A), D31.1 (K), D32.2 (A), D41.1 (K), D42.2 (A), D51.1 (K), D52.2 (A), D61.1 (K), D62.2 (A), D71.1 (K), D72.2 (A), D81.1 (K), D82.2 (A); no longer D3.2 (A)
- net +3V3: now also D3.2 (A), C10.1, U10.10 (V3), U10.7 (VCC)
- net +5V: now also J10.A4 (VBUS), J10.A9 (VBUS), J10.B4 (VBUS), J10.B9 (VBUS)
- net GND: now also R3.2, R4.2, R5.2, R6.2, R7.2, C10.2, J10.A1 (GND), J10.A12 (GND), J10.B1 (GND), J10.B12 (GND), R11.2, R21.2, R31.2, R41.2, R51.2, R61.2, R71.2, R81.2, U10.3 (GND)
- net GNDPWR: now also C9.2, Q1.2 (E), Q2.2 (E), Q3.2 (E), Q4.2 (E), Q5.2 (E), Q6.2 (E), Q7.2 (E), Q8.2 (E), R12.2, R22.2, R32.2, R42.2, R52.2, R62.2, R72.2, R82.2
- net GPIO1: now also U11.6 (PA0), U1.1
- net GPIO2: now also U11.7 (PA1), U2.1
- net GPIO3: now also U11.9 (PA3), U3.1
- net GPIO4: now also U11.10 (PA4), U4.1
- net GPIO5: now also U11.11 (PA5), U5.1
- net GPIO6: now also U11.12 (PA6), U6.1
- net GPIO7: now also U11.13 (PA7), U7.1
- net GPIO8: now also U11.18 (PA8), U8.1
- net at R4.1: now also R5.1, J10.A5 (CC1)
- net at R6.1: now also R7.1, J10.B5 (CC2)
- net USART1_TX: now reaches U11.19 (PA9)
- net USART1_RX: now reaches U11.20 (PA10)
- net OUT1: no longer names the net of D11.2 (A), J1.1 (Pin_1)
- net OUT1: now also Q1.3 (C), R14.2, U1.4; no longer R13.2
- net OUT2: no longer names the net of J2.1 (Pin_1)
- net OUT2: now also D21.2 (A), Q2.3 (C), R24.2, U2.4
- net OUT3: no longer names the net of J3.1 (Pin_1)
- net OUT3: now also D31.2 (A), Q3.3 (C), R34.2, U3.4; no longer R3.2
- net OUT4: no longer names the net of J4.1 (Pin_1)
- net OUT4: now also D41.2 (A), Q4.3 (C), R44.2, U4.4; no longer R4.2
- net OUT5: no longer names the net of J5.1 (Pin_1)
- net OUT5: now also D51.2 (A), Q5.3 (C), R54.2, U5.4; no longer R5.2
- net OUT6: no longer names the net of J6.1 (Pin_1)
- net OUT6: now also D61.2 (A), Q6.3 (C), R64.2, U6.4; no longer R6.2
- net OUT7: no longer names the net of J7.1 (Pin_1)
- net OUT7: now also D71.2 (A), Q7.3 (C), R74.2, U7.4; no longer R7.2
- net OUT8: no longer names the net of J8.1 (Pin_1)
- net OUT8: now also D81.2 (A), Q8.3 (C), R84.2, U8.4
- new net: Q5.1 (B), R52.1, U5.3
- new net: R61.1, U6.2
- new net: Q3.1 (B), R32.1, U3.3
- new net: Q7.1 (B), R72.1, U7.3
- new net: R81.1, U8.2
- new net: R71.1, U7.2
- new net: R31.1, U3.2
- new net: Q8.1 (B), R82.1, U8.3
- new net: R83.2, R84.1
- new net: Q1.1 (B), R12.1, U1.3
- new net: Q6.1 (B), R62.1, U6.3
- new net: D52.1 (K), R53.1
- new net: R51.1, U5.2
- new net: Q4.1 (B), R42.1, U4.3
- new net: D32.1 (K), R33.1
- new net: D22.1 (K), R23.1
- new net: R23.2, R24.1
- new net: D62.1 (K), R63.1
- new net: R63.2, R64.1
- new net: Q2.1 (B), R22.1, U2.3
- new net: R13.2, R14.1
- new net: R53.2, R54.1
- new net: R73.2, R74.1
- new net: J10.A6 (D+), J10.B6 (D+), U10.1 (UD+)
- new net: J10.A7 (D-), J10.B7 (D-), U10.2 (UD-)
- new net: R33.2, R34.1
- new net: R11.1, U1.2
- new net: R41.1, U4.2
- new net: D82.1 (K), R83.1
- new net: D42.1 (K), R43.1
- new net: D72.1 (K), R73.1
- new net: R43.2, R44.1
- new net: R21.1, U2.2
- new net USARTx_RX: U10.8 (TXD)
- new net USARTx_TX: U10.9 (RXD)
- no-connect marks 21 -> 24
Other:
- note added: "NJM12877F33"
- moved on the sheet: C2, C3, C4, C5, C6, D11, D12, J1, J12, J9, R13, U9

Commit message: chore: Update Air.kicad_pro configuration file
Connections:
- net USARTx_RX is gone; now on net VCP_RX: U10.8 (TXD)
- net USARTx_TX is gone; now on net VCP_TX: U10.9 (RXD)
Changed lines of the file:
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@@
 		)
 	)
-	(global_label "USARTx_RX"
+	(global_label "VCP_RX"
 		(shape output)
 		(at 516.89 147.32 0)
@@
 		)
 		(property "Intersheetrefs" "${INTERSHEET_REFS}"
-			(at 529.7402 147.32 0)
+			(at 526.9509 147.32 0)
 			(effects
 				(font
@@
 		)
 	)
-	(global_label "USARTx_TX"
+	(global_label "VCP_TX"
 		(shape input)
 		(at 516.89 149.86 0)
@@
 		)
 		(property "Intersheetrefs" "${INTERSHEET_REFS}"
-			(at 529.4378 149.86 0)
+			(at 526.6485 149.86 0)
 			(effects
 				(font
@@
 		)
 		(instances
-			(project ""
+			(project "Air"
 				(path "/9538e4ed-27e6-4c37-b989-9859dc0d49e8"
 					(reference "#PWR030")
@@
 		)
 		(instances
-			(project ""
+			(project "Air"
 				(path "/9538e4ed-27e6-4c37-b989-9859dc0d49e8"
 					(reference "#PWR048")
@@
 		)
 		(instances
-			(project ""
+			(project "Air"
 				(path "/9538e4ed-27e6-4c37-b989-9859dc0d49e8"
 					(reference "#PWR022")
@@
 		)
 		(instances
-			(project ""
+			(project "Air"
 				(path "/9538e4ed-27e6-4c37-b989-9859dc0d49e8"
 					(reference "#PWR04")
@@
 		)
 		(instances
-			(project ""
+			(project "Air"
 				(path "/9538e4ed-27e6-4c37-b989-9859dc0d49e8"
 					(reference "#PWR021")
@@
 		)
 		(instances
-			(project ""
+			(project "Air"
 				(path "/9538e4ed-27e6-4c37-b989-9859dc0d49e8"
 					(reference "#PWR028")
@@
 		)
 		(instances
-			(project ""
+			(project "Air"
 				(path "/9538e4ed-27e6-4c37-b989-9859dc0d49e8"
 					(reference "#PWR09")
@@
 		)
 		(instances
-			(project ""
+			(project "Air"
 				(path "/9538e4ed-27e6-4c37-b989-9859dc0d49e8"
 					(reference "#FLG06")
@@
 		)
 		(instances
-			(project ""
+			(project "Air"
 				(path "/9538e4ed-27e6-4c37-b989-9859dc0d49e8"
 					(reference "C5")
@@
 		)
 		(instances
-			(project ""
+			(project "Air"
 				(path "/9538e4ed-27e6-4c37-b989-9859dc0d49e8"
 					(reference "#PWR02")
@@
 		)
 		(instances
-			(project ""
+			(project "Air"
 				(path "/9538e4ed-27e6-4c37-b989-9859dc0d49e8"
 					(reference "#PWR029")
@@
 		)
 		(instances
-			(project ""
+			(project "Air"
 				(path "/9538e4ed-27e6-4c37-b989-9859dc0d49e8"
 					(reference "R2")
@@
 		)
 		(instances
-			(project ""
+			(project "Air"
 				(path "/9538e4ed-27e6-4c37-b989-9859dc0d49e8"
 					(reference "U12")
@@
 		)
 		(instances
-			(project ""
+			(project "Air"
 				(path "/9538e4ed-27e6-4c37-b989-9859dc0d49e8"
 					(reference "#FLG01")
@@
 		)
 		(instances
-			(project ""
+			(project "Air"
 				(path "/9538e4ed-27e6-4c37-b989-9859dc0d49e8"
 					(reference "#PWR06")
@@
 		)
 		(instances
-			(project ""
+			(project "Air"
 				(path "/9538e4ed-27e6-4c37-b989-9859dc0d49e8"
 					(reference "J1")
@@
 		)
 		(instances
-			(project ""
+			(project "Air"
 				(path "/9538e4ed-27e6-4c37-b989-9859dc0d49e8"
 					(reference "D3")
@@
 		)
 		(instances
-			(project ""
+			(project "Air"
 				(path "/9538e4ed-27e6-4c37-b989-9859dc0d49e8"
 					(reference "#FLG05")
@@
 		)
 		(instances
-			(project ""
+			(project "Air"
 				(path "/9538e4ed-27e6-4c37-b989-9859dc0d49e8"
 					(reference "Q1")
@@
 		)
 		(instances
-			(project ""
+			(project "Air"
 				(path "/9538e4ed-27e6-4c37-b989-9859dc0d49e8"
 					(reference "C9")
@@
 	)
 	(symbol
+		(lib_name "LED_5")
 		(lib_id "Device:LED")
 		(at 335.28 -118.11 90)
@@
 		)
 		(instances
-			(project ""
+			(project "Air"
 				(path "/9538e4ed-27e6-4c37-b989-9859dc0d49e8"
 					(reference "#PWR03")
@@
 	)
 	(symbol
+		(lib_name "LED_3")
 		(lib_id "Device:LED")
 		(at 193.04 -118.11 90)
@@
 	)
 	(symbol
+		(lib_name "LED_2")
 		(lib_id "Device:LED")
 		(at 121.92 -118.11 90)
@@
 		)
 		(instances
-			(project ""
+			(project "Air"
 				(path "/9538e4ed-27e6-4c37-b989-9859dc0d49e8"
 					(reference "R13")
@@
 		)
 		(instances
-			(project ""
+			(project "Air"
 				(path "/9538e4ed-27e6-4c37-b989-9859dc0d49e8"
 					(reference "J9")
@@
 		)
 		(instances
-			(project ""
+			(project "Air"
 				(path "/9538e4ed-27e6-4c37-b989-9859dc0d49e8"
 					(reference "#PWR049")
@@
 		)
 		(instances
-			(project ""
+			(project "Air"
 				(path "/9538e4ed-27e6-4c37-b989-9859dc0d49e8"
 					(reference "#PWR027")
@@
 		)
 		(instances
-			(project ""
+			(project "Air"
 				(path "/9538e4ed-27e6-4c37-b989-9859dc0d49e8"
 					(reference "#PWR047")
@@
 		)
 		(instances
-			(project ""
+			(project "Air"
 				(path "/9538e4ed-27e6-4c37-b989-9859dc0d49e8"
 					(reference "#PWR043")
@@
 		)
 		(instances
-			(project ""
+			(project "Air"
 				(path "/9538e4ed-27e6-4c37-b989-9859dc0d49e8"
 					(reference "#PWR044")
@@
 		)
 		(instances
-			(project ""
+			(project "Air"
 				(path "/9538e4ed-27e6-4c37-b989-9859dc0d49e8"
 					(reference "U10")
@@
 		)
 		(instances
-			(project ""
+			(project "Air"
 				(path "/9538e4ed-27e6-4c37-b989-9859dc0d49e8"
 					(reference "#PWR0102")
@@
 		)
 		(instances
-			(project ""
+			(project "Air"
 				(path "/9538e4ed-27e6-4c37-b989-9859dc0d49e8"
 					(reference "#PWR046")
@@
 		)
 		(instances
-			(project ""
+			(project "Air"
 				(path "/9538e4ed-27e6-4c37-b989-9859dc0d49e8"
 					(reference "#PWR01")
@@
 		)
 		(instances
-			(project ""
+			(project "Air"
 				(path "/9538e4ed-27e6-4c37-b989-9859dc0d49e8"
 					(reference "R11")
@@
 		)
 		(instances
-			(project ""
+			(project "Air"
 				(path "/9538e4ed-27e6-4c37-b989-9859dc0d49e8"
 					(reference "C2")
@@
 	)
 	(symbol
+		(lib_name "LED_8")
 		(lib_id "Device:LED")
 		(at 548.64 -118.11 90)
@@
 		)
 		(instances
-			(project ""
+			(project "Air"
 				(path "/9538e4ed-27e6-4c37-b989-9859dc0d49e8"
 					(reference "J12")
@@
 		)
 		(instances
-			(project ""
+			(project "Air"
 				(path "/9538e4ed-27e6-4c37-b989-9859dc0d49e8"
 					(reference "R12")
@@
 		)
 		(instances
-			(project ""
+			(project "Air"
 				(path "/9538e4ed-27e6-4c37-b989-9859dc0d49e8"
 					(reference "#PWR045")
@@
 	)
 	(symbol
+		(lib_name "LED_4")
 		(lib_id "Device:LED")
 		(at 264.16 -118.11 90)
@@
 		)
 		(instances
-			(project ""
+			(project "Air"
 				(path "/9538e4ed-27e6-4c37-b989-9859dc0d49e8"
 					(reference "J10")
@@
 	)
 	(symbol
+		(lib_name "LED_7")
 		(lib_id "Device:LED")
 		(at 477.52 -118.11 90)
@@
 		)
 		(instances
-			(project ""
+			(project "Air"
 				(path "/9538e4ed-27e6-4c37-b989-9859dc0d49e8"
 					(reference "U1")
@@
 		)
 		(instances
-			(project ""
+			(project "Air"
 				(path "/9538e4ed-27e6-4c37-b989-9859dc0d49e8"
 					(reference "R3")
@@
 		)
 		(instances
-			(project ""
+			(project "Air"
 				(path "/9538e4ed-27e6-4c37-b989-9859dc0d49e8"
 					(reference "C1")
@@
 		)
 		(instances
-			(project ""
+			(project "Air"
 				(path "/9538e4ed-27e6-4c37-b989-9859dc0d49e8"
 					(reference "SW1")
@@
 	)
 	(symbol
+		(lib_name "LED_1")
 		(lib_id "Device:LED")
 		(at 50.8 -118.11 90)
@@
 		)
 		(instances
-			(project ""
+			(project "Air"
 				(path "/9538e4ed-27e6-4c37-b989-9859dc0d49e8"
 					(reference "D12")
@@
 		)
 		(instances
-			(project ""
+			(project "Air"
 				(path "/9538e4ed-27e6-4c37-b989-9859dc0d49e8"
 					(reference "J11")
@@
 		)
 		(instances
-			(project ""
+			(project "Air"
 				(path "/9538e4ed-27e6-4c37-b989-9859dc0d49e8"
 					(reference "#PWR025")
@@
 		)
 		(instances
-			(project ""
+			(project "Air"
 				(path "/9538e4ed-27e6-4c37-b989-9859dc0d49e8"
 					(reference "#PWR020")
@@
 		)
 		(instances
-			(project ""
+			(project "Air"
 				(path "/9538e4ed-27e6-4c37-b989-9859dc0d49e8"
 					(reference "#PWR010")
@@
 	)
 	(symbol
+		(lib_name "LED_6")
 		(lib_id "Device:LED")
 		(at 406.4 -118.11 90)
@@
 		)
 		(instances
-			(project ""
+			(project "Air"
 				(path "/9538e4ed-27e6-4c37-b989-9859dc0d49e8"
 					(reference "#PWR05")
@@
 		)
 		(instances
-			(project ""
+			(project "Air"
 				(path "/9538e4ed-27e6-4c37-b989-9859dc0d49e8"
 					(reference "#PWR026")
@@
 		)
 		(instances
-			(project ""
+			(project "Air"
 				(path "/9538e4ed-27e6-4c37-b989-9859dc0d49e8"
 					(reference "#PWR050")
@@
 		)
 		(instances
-			(project ""
+			(project "Air"
 				(path "/9538e4ed-27e6-4c37-b989-9859dc0d49e8"
 					(reference "D11")
@@
 		)
 		(instances
-			(project ""
+			(project "Air"
 				(path "/9538e4ed-27e6-4c37-b989-9859dc0d49e8"
 					(reference "R5")
@@
 		)
 		(instances
-			(project ""
+			(project "Air"
 				(path "/9538e4ed-27e6-4c37-b989-9859dc0d49e8"
 					(reference "C10")
@@
 		)
 		(instances
-			(project ""
+			(project "Air"
 				(path "/9538e4ed-27e6-4c37-b989-9859dc0d49e8"
 					(reference "U11")
@@
 		)
 		(instances
-			(project ""
+			(project "Air"
 				(path "/9538e4ed-27e6-4c37-b989-9859dc0d49e8"
 					(reference "U9")
